Commit message: udev rules

File: ros2_ws/src/robot_bringup/urdf/robot.urdf.xacro (robot description, xacro)
@@ -5,7 +5,7 @@
     <visual>
       <geometry>
-        <box size="0.4 0.3 0.1"/>
+        <box size="0.32 0.29 0.2"/>
       </geometry>
-      <origin xyz="0 0 0.05"/>
+      <origin xyz="0 0 0"/>
     </visual>
   </link>
@@ -15,5 +15,5 @@
     <parent link="base_link"/>
     <child link="left_wheel_link"/>
-    <origin xyz="0.0 0.15 0.0" rpy="0 0 0"/>
+    <origin xyz="0.0 0.12 0.0" rpy="0 0 0"/>
     <axis xyz="0 1 0"/>
   </joint>
@@ -23,5 +23,5 @@
     <parent link="base_link"/>
     <child link="right_wheel_link"/>
-    <origin xyz="0.0 -0.15 0.0" rpy="0 0 0"/>
+    <origin xyz="0.0 -0.12 0.0" rpy="0 0 0"/>
     <axis xyz="0 1 0"/>
   </joint>

Commit message: nav 2

File: ros2_ws/src/robot_bringup/urdf/robot.urdf.xacro (robot description, xacro)
@@ -10,20 +10,4 @@
     </visual>
   </link>
-  <!-- Left Wheel -->
-  <link name="left_wheel_link"/>
-  <joint name="left_wheel_joint" type="continuous">
-    <parent link="base_link"/>
-    <child link="left_wheel_link"/>
-    <origin xyz="0.0 0.12 0.0" rpy="0 0 0"/>
-    <axis xyz="0 1 0"/>
-  </joint>
-  <!-- Right Wheel -->
-  <link name="right_wheel_link"/>
-  <joint name="right_wheel_joint" type="continuous">
-    <parent link="base_link"/>
-    <child link="right_wheel_link"/>
-    <origin xyz="0.0 -0.12 0.0" rpy="0 0 0"/>
-    <axis xyz="0 1 0"/>
-  </joint>
   <!-- IMU -->
   <link name="imu_link"/>
@@ -47,24 +31,3 @@
     <origin xyz="0 0 0.2" rpy="0 0 0"/>
   </joint>
-  <!-- ros2_control interface -->
-  <ros2_control name="RoboClawSystem" type="system">
-    <hardware>
-      <plugin>roboclaw_hardware_interface/RoboClawHardwareInterface</plugin>
-      <param name="serial_port">/dev/roboclaw</param>
-    </hardware>
-    <joint name="left_wheel_joint">
-      <command_interface name="velocity"/>
-      <state_interface name="position"/>
-      <param name="address">128</param>
-      <param name="qppr">6533</param>
-      <param name="motor_type">M2</param>
-    </joint>
-    <joint name="right_wheel_joint">
-      <command_interface name="velocity"/>
-      <state_interface name="position"/>
-      <param name="address">128</param>
-      <param name="qppr">6533</param>
-      <param name="motor_type">M1</param>
-    </joint>
-  </ros2_control>
 </robot>

Commit message: urdf

File: ros2_ws/src/robot_bringup/urdf/robot.urdf.xacro (robot description, xacro)
@@ -15,5 +15,5 @@
     <parent link="base_link"/>
     <child link="imu_link"/>
-    <origin xyz="0 0 0.1" rpy="0 0 0"/>
+    <origin xyz="-0.07 0.03 0.05" rpy="0 0 3.1416"/>
   </joint>
   <!-- GPS -->
@@ -22,5 +22,5 @@
     <parent link="base_link"/>
     <child link="gps_link"/>
-    <origin xyz="0 0 0.15" rpy="0 0 0"/>
+    <origin xyz="0 -0.06 0.185" rpy="0 0 1.57"/>
   </joint>
   <!-- Lidar -->
@@ -29,5 +29,5 @@
     <parent link="base_link"/>
     <child link="lidar_link"/>
-    <origin xyz="0 0 0.2" rpy="0 0 0"/>
+    <origin xyz="0 0 0.21" rpy="0 0 0"/>
   </joint>
 </robot>

Commit message: small fix

File: ros2_ws/src/robot_bringup/urdf/robot.urdf.xacro (robot description, xacro)
@@ -15,5 +15,5 @@
     <parent link="base_link"/>
     <child link="imu_link"/>
-    <origin xyz="-0.07 0.03 0.05" rpy="0 0 3.1416"/>
+    <origin xyz="-0.07 0.03 0.05" rpy="0 0 0"/>
   </joint>
   <!-- GPS -->

Commit message: covariance turning

File: ros2_ws/src/robot_bringup/urdf/robot.urdf.xacro (robot description, xacro)
@@ -15,5 +15,5 @@
     <parent link="base_link"/>
     <child link="imu_link"/>
-    <origin xyz="-0.07 0.03 0.05" rpy="0 0 0"/>
+    <origin xyz="-0.07 0.0 0.05" rpy="0 0 0"/>
   </joint>
   <!-- GPS -->
@@ -22,5 +22,5 @@
     <parent link="base_link"/>
     <child link="gps_link"/>
-    <origin xyz="0 -0.06 0.185" rpy="0 0 1.57"/>
+    <origin xyz="0.0 0.05 0.05" rpy="0 0 0"/>
   </joint>
   <!-- Lidar -->

Commit message: Update robot bringup geometry and nav2 navigation parameters

File: ros2_ws/src/robot_bringup/urdf/robot.urdf.xacro (robot description, xacro)
@@ -5,5 +5,5 @@
     <visual>
       <geometry>
-        <box size="0.32 0.29 0.2"/>
+        <box size="0.4 0.37 0.17"/>
       </geometry>
       <origin xyz="0 0 0"/>
